File: gameconsole/gameconsole.kicad_sch (KiCad schematic)
At the start: 110 parts, among them J1 62684-401100ALF, J2 USB4216-03-A_REVA, J3 NTCLE413E2103F520L, J4 S2B-PH-K-S_LF__SN_, J5 S2B-XH-A_LF__SN_, SW1 PTS810 (250gf), SW2 PTS810 (250gf), SW3 SW_Push, U1 ESP32-S3-WROOM-1, U2 BQ25895RTWR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

Commit message: PCB Drawings
Parts:
- C16: value 1uF -> 10nF; footprint Capacitor_SMD:C_0805_2012Metric_Pad1.18x1.45mm_HandSolder -> GRM1885C1H103JA01D:CAPC1608X90N; Description_1 1uF, 16V or higher, X7R, 0805 -> 10nF, 16V or higher, X7R, 0805
