File: gameconsole/gameconsole.kicad_pcb (KiCad board)
At the start: 4 copper layers, 234.1 x 105.6 mm, 118 parts, among them J1 62684-401100ALF, J2 USB4216-03-A_REVA, J3 NTCLE413E2103F520L, J4 S2B-PH-K-S_LF__SN_, J5 S2B-XH-A_LF__SN_, SW1 PTS810 (250gf), SW2 PTS810 (250gf), SW3 SW_Push, U1 ESP32-S3-WROOM-1, U2 BQ25895RTWR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

Commit message: Revised Gameconsole kicad schematic
Parts:
- moved L3 25.6 mm to (102.8, 97.8), turned to 180 degrees
- moved D2 25.3 mm to (111.2, 99.5), turned to 0 degrees
- moved C25 24.9 mm to (94.3, 101.5), turned to -90 degrees
- moved C26 20.2 mm to (96.9, 101.5), turned to -90 degrees
- moved R26 19.1 mm to (102.0, 107.8), turned to 0 degrees
- moved R29 10.9 mm to (101.5, 103.2), turned to 180 degrees
- moved R27 10.1 mm to (106.0, 107.8), turned to 0 degrees
- moved R28 9.76 mm to (109.0, 108.8), turned to -90 degrees
- moved C28 8.47 mm to (105.5, 105.5), turned to 180 degrees
- moved R25 7.87 mm to (113.5, 109.2)
- moved R24 6.83 mm to (117.0, 104.5), turned to 180 degrees
- moved C24 4.71 mm to (113.1, 107.5), turned to 0 degrees
- moved C27 4.23 mm to (105.5, 103.2), turned to 180 degrees
- moved C20 2.77 mm to (109.5, 97.0)
Routing:
- net PH: track 46.7 -> 0.00 mm
- net ADDR: track 331.2 -> 302.6 mm
- net BTNPU: track 474.8 -> 490.5 mm
- net PWR: track 98.3 -> 86.9 mm
- net Net-(U7-COMP): track 15.3 -> 4.65 mm
- net VSNS: track 14.5 -> 4.00 mm
- net BOOT: track 3.55 -> 10.6 mm
- net EN: track 14.5 -> 7.92 mm
- net Net-(R26-Pad2): track 5.59 -> 2.00 mm
- net SS: track 4.17 -> 1.69 mm
- net Net-(C27-Pad2): track 4.17 -> 1.96 mm
- net GAIN_SLOT: track 66.9 -> 65.6 mm
- net SFXBCLK: track 56.5 -> 57.4 mm
- net D+: track 81.5 -> 80.8 mm
- added copper zone on B.Cu, net ADDR
- added copper zone on B.Cu, net BTNPU
- added copper zone on B.Cu, net PH
- added copper zone on B.Cu, net PWR

Commit message: PCB Drawings
Parts:
- C16: value 1uF -> 10nF; footprint Capacitor_SMD:C_0805_2012Metric_Pad1.18x1.45mm_HandSolder -> GRM1885C1H103JA01D:CAPC1608X90N
- R11: value 10K -> 10k
- moved R43 88.4 mm to (102.2, 75.2), turned to 90 degrees
- moved R41 40.0 mm to (236.0, 85.8), turned to 90 degrees
- moved R33 36.5 mm to (233.8, 85.8), turned to 90 degrees
- moved R32 34.8 mm to (238.2, 92.8)
- moved R37 31.7 mm to (243.2, 92.8), turned to -90 degrees
- moved R36 31.5 mm to (240.8, 92.8), turned to -90 degrees
- moved R39 27.7 mm to (231.5, 85.8), turned to 90 degrees
- moved R34 27.2 mm to (240.8, 85.8), turned to 90 degrees
- moved R47 26.4 mm to (99.5, 80.8), turned to 180 degrees
- moved R35 25.4 mm to (243.2, 85.8), turned to 90 degrees
- moved R38 24.5 mm to (238.2, 85.8)
- moved R46 23.9 mm to (99.2, 78.0), turned to 180 degrees
- moved C23 12.0 mm to (122.0, 106.0)
- moved R4 8.23 mm to (195.5, 114.8), turned to 0 degrees
- moved C5 6.57 mm to (117.6, 112.1)
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Routing:
- net BTNPU: track 490.5 -> 354.2 mm
- net PWR: track 86.9 -> 6.50 mm
- net Net-(U4-P14): track 77.1 -> 107.6 mm
- net ADDR: track 302.6 -> 272.3 mm
- net Net-(U4-P15): track 65.9 -> 92.1 mm
- net Net-(U4-P17): track 92.9 -> 109.8 mm, vias 2 -> 1
- net Net-(U4-P23): track 219.4 -> 232.3 mm
- net Net-(U4-P03): track 92.6 -> 104.8 mm
- net Net-(U4-P02): track 85.5 -> 94.1 mm
- net Net-(U4-P24): track 210.3 -> 216.2 mm
- net Net-(U4-P00): track 103.3 -> 109.0 mm
- net Net-(U4-P04): track 74.8 -> 79.8 mm
- net INTPWR: track 112.2 -> 116.1 mm
- net Net-(U4-P27): track 191.0 -> 194.8 mm
- net STATPWR: track 104.5 -> 108.2 mm
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- added copper zone on F.Cu, net PWR

Commit message: Add files via upload
Routing:
- net BTNPU: track 354.2 -> 335.5 mm
- net ADDR: track 272.3 -> 273.1 mm, vias 100 -> 103
Changed lines of the file:
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@@
+	)
+	(via
+		(at 111.5 105.25)
+		(size 0.6)
+		(drill 0.3)
+		(layers "F.Cu" "B.Cu")
+		(net "ADDR")
 	)
 	(via
@@
 	(via
 		(at 44.5 75.06)
+		(size 0.6)
+		(drill 0.3)
+		(layers "F.Cu" "B.Cu")
+		(net "ADDR")
+	)
+	(via
+		(at 111.75 102.25)
 		(size 0.6)
 		(drill 0.3)
@@
 	)
 	(via
+		(at 111.25 104.25)
+		(size 0.6)
+		(drill 0.3)
+		(layers "F.Cu" "B.Cu")
+		(net "ADDR")
+	)
+	(via
 		(at 96.75 105.5)
 		(size 0.6)
@@
 	)
 	(segment
+		(start 111.75 102)
+		(end 111.75 102.25)
+		(width 0.2)
+		(layer "B.Cu")
+		(net "ADDR")
+	)
+	(segment
 		(start 152.6715 86.7195)
 		(end 152.3715 86.7195)
@@
 	)
 	(segment
+		(start 111.75 105)
+		(end 111.5 105.25)
+		(width 0.2)
+		(layer "B.Cu")
+		(net "ADDR")
+	)
+	(segment
 		(start 128.7715 93.5395)
 		(end 128.3115 93.9995)
@@
 	)
 	(segment
+		(start 111.25 104)
+		(end 111.25 104.25)
+		(width 0.2)
+		(layer "B.Cu")
+		(net "ADDR")
+	)
+	(segment
 		(start 100.5 103.25)
 		(end 99 103.25)
@@
 	)
 	(segment
-		(start 82.7255 101.5455)
-		(end 82.4855 101.7855)
-		(width 2)
-		(layer "B.Cu")
-		(net "BTNPU")
-	)
-	(segment
 		(start 125.2295 122.5795)
 		(end 125.97 123.32)
@@
 	)
 	(segment
-		(start 82.7255 101.5455)
-		(end 83 101.271)
-		(width 2)
-		(layer "B.Cu")
-		(net "BTNPU")
-	)
-	(segment
 		(start 148.3315 101.9695)
 		(end 150.2015 103.8395)
@@
 	)
 	(segment
-		(start 79.7615 104.5095)
-		(end 79.7615 113.9595)
-		(width 2)
-		(layer "B.Cu")
-		(net "BTNPU")
-	)
-	(segment
 		(start 92.25 95.75)
 		(end 92.25 96)
@@
 	)
 	(segment
-		(start 82.7255 101.5455)
-		(end 79.7615 104.5095)
-		(width 2)
-		(layer "B.Cu")
-		(net "BTNPU")
-	)
-	(segment
 		(start 150.4115 99.8895)
 		(end 150.4815 99.8895)
@@
 	)
 	(segment
+		(start 90.3855 108.8855)
+		(end 110.99 129.49)
+		(width 2)
+		(layer "B.Cu")
+		(net "BTNPU")
+	)
+	(segment
 		(start 115.451 129.49)
 		(end 118.0015 126.9395)
@@
 	)
 	(segment
+		(start 90.3855 93.8855)
+		(end 90.3855 108.8855)
+		(width 2)
+		(layer "B.Cu")
+		(net "BTNPU")
+	)
+	(segment
 		(start 202.2715 105.2195)
 		(end 193.6715 113.8195)
@@
 	)
 	(segment
+		(start 110.99 129.49)
+		(end 111.7 129.49)
+		(width 2)
+		(layer "B.Cu")
+		(net "BTNPU")
+	)
+	(segment
 		(start 151.8965 93.0445)
 		(end 153.1515 91.7895)
@@
 	)
 	(segment
-		(start 79.7615 113.9595)
-		(end 95.292 129.49)
-		(width 2)
-		(layer "B.Cu")
-		(net "BTNPU")
-	)
-	(segment
 		(start 202.2715 101.0215)
 		(end 202.2715 103.5)
@@
 		(width 2)
 		(layer "B.Cu")
-		(net "BTNPU")
-	)
-	(segment
-		(start 95.292 129.49)
-		(end 111.7 129.49)
-		(width 2)
-		(layer "B.Cu")
-		(net "BTNPU")
-	)
-	(segment
-		(start 82.7255 101.5455)
-		(end 90.3855 93.8855)
-		(width 2)
-		(layer "B.Cu")
